File: roadrunner/roadrunner.kicad_pcb (KiCad board)
At the start: 2 copper layers, 246.8 x 97.3 mm, 87 parts, among them J1 Battery_conn, J2 battery_conn_r, J3 Conn_01x12_Female, J4 niceview_left, J5 niceview_right, SW1 SW_Push, SW10 SW_Push, SW10_r1 SW_Push, SW11 SW_Push, SW11_r1 SW_Push, SW12 SW_Push, SW12_r1 SW_Push, SW13 SW_Push, SW13_r1 SW_Push, SW14 SW_Push, SW14_r1 SW_Push, SW15 SW_Push, SW15_r1 SW_Push, SW16 SW_Push, SW16_r1 SW_Push, SW17 SW_Push, SW17_r1 SW_Push, SW1_r1 SW_Push, SW2 SW_Push, SW2_r1 SW_Push, SW3 SW_Push, SW3_r1 SW_Push, SW4 SW_Push, SW4_r1 SW_Push, SW5 SW_Push, SW5_r1 SW_Push, SW6 SW_Push, SW6_r1 SW_Push, SW7 SW_Push, SW7_r1 SW_Push, SW8 SW_Push, SW8_r1 SW_Push, SW9 SW_Push, SW9_r1 SW_Push, U1 ProMicro-kbd, U2 ProMicro-kbd

Commit message: feat: add vik
Parts:
- added J6: track_point_right, Connector_FFC-FPC:TE_1-84953-2_1x12-1MP_P1.0mm_Horizontal, B.Cu at (116.3, 34.6)
- added J7: VIK_Left, Connector_FFC-FPC:Hirose_FH12-12S-0.5SH_1x12-1MP_P0.50mm_Horizontal, F.Cu at (266.8, 75.7)
- added J8: VIK_Right, Connector_FFC-FPC:Hirose_FH12-12S-0.5SH_1x12-1MP_P0.50mm_Horizontal, F.Cu at (28.8, 75.8)
- J3: value Conn_01x12_Female -> track_point_left; footprint Connector_FFC-FPC:Hirose_FH12-12S-0.5SH_1x12-1MP_P0.50mm_Horizontal -> Connector_FFC-FPC:TE_1-84953-2_1x12-1MP_P1.0mm_Horizontal
- moved J3 65.4 mm to (180.3, 34.9)
- moved D23 2.16 mm to (76.6, 60.0)
- moved D19 1.34 mm to (64.3, 53.1)
- moved RSW2 1.00 mm to (49.7, 87.9)
Connections:
- J3 pad 1: VCC -> vcc
- J3 pad 2: GND -> IPD_DATA
- J3 pad 3: IPD_CLK -> IPD_RST
- J3 pad 7: IPD_RST -> gnd
- J3 pad 8: IPD_DATA -> IPD_CLK
- U1 pad 18: unconnected-(U1-Pad18) -> GPIO1
- U1 pad 19: unconnected-(U1-Pad19) -> IPD_RST
- U1 pad 2: unconnected-(U1-Pad2) -> MISO
- U1 pad 20: unconnected-(U1-Pad20) -> GPIO2
- U1 pad 7: unconnected-(U1-Pad7) -> IPD_DATA
- U1 pad 8: unconnected-(U1-Pad8) -> IPD_CLK
- U2 pad 1: CS_R -> CS_r
- U2 pad 18: unconnected-(U2-Pad18) -> GPIO1_r
- U2 pad 19: unconnected-(U2-Pad19) -> IPD_RST_r
- U2 pad 2: unconnected-(U2-Pad2) -> MISO_r
- U2 pad 20: unconnected-(U2-Pad20) -> GPIO2_r
- U2 pad 7: unconnected-(U2-Pad7) -> IPD_DATA_r
- U2 pad 8: unconnected-(U2-Pad8) -> IPD_CLK_r
Other:
- outline, holes or cut-outs redrawn

Commit message: update thumbpoint layout
Parts:
- moved SW_POWERR1 0.12 mm to (40.8, 50.3)
Other:
- outline, holes or cut-outs redrawn

Commit message: feat: begin routing
Parts:
- moved D29 1.28 mm to (65.7, 88.6), turned to 180 degrees
- moved D24 1.21 mm to (65.9, 71.8), turned to 180 degrees
- moved D25 1.11 mm to (93.2, 53.3), turned to 180 degrees
- moved D32 0.96 mm to (129.4, 89.0), turned to 180 degrees
- moved D33 0.94 mm to (56.0, 111.3), turned to 180 degrees
- moved D30 0.90 mm to (93.3, 70.4), turned to 180 degrees
- moved D27 0.83 mm to (129.2, 72.0), turned to 180 degrees
- moved D34 0.80 mm to (74.9, 104.6), turned to 180 degrees
- moved D31 0.79 mm to (111.4, 77.1), turned to 180 degrees
- moved D20 0.61 mm to (93.2, 35.8), turned to 180 degrees
- moved D18 0.55 mm to (75.1, 41.4), turned to 180 degrees
- moved D22 0.45 mm to (129.1, 54.9), turned to 180 degrees
- moved D28 0.43 mm to (75.3, 75.6), turned to 180 degrees
- moved D26 0.38 mm to (111.5, 60.2), turned to 180 degrees
- moved D21 0.32 mm to (111.1, 42.7), turned to 180 degrees
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Routing:
- net COL4_r: track 0.00 -> 153.4 mm
- net ROW2_r: track 0.00 -> 111.4 mm
- net COL3_r: track 0.00 -> 102.1 mm, vias 0 -> 4
- net ROW1_r: track 0.00 -> 99.5 mm
- net ROW0_r: track 0.00 -> 96.3 mm
- net vcc_r: track 0.00 -> 80.3 mm, vias 0 -> 3
- net IPD_RST_r: track 0.00 -> 78.6 mm, vias 0 -> 2
- net IPD_DATA_r: track 0.00 -> 76.2 mm, vias 0 -> 2
- net COL2_r: track 0.00 -> 74.0 mm, vias 0 -> 4
- net IPD_CLK_r: track 0.00 -> 71.5 mm, vias 0 -> 2
- net gnd_r: track 0.00 -> 70.1 mm, vias 0 -> 2
- net COL1_r: track 0.00 -> 57.7 mm, vias 0 -> 4
- net COL0_r: track 0.00 -> 34.3 mm, vias 0 -> 4
- net ROW3_r: track 0.00 -> 22.0 mm
- net Net-(D29-A): track 0.00 -> 15.1 mm
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
Commit message: add traces
Parts:
- removed REF_PUCK_R, e: Tenting Puck, * duckyb-collection:Tenting_Puck2_no_pads
- moved D2 2.78 mm to (176.0, 45.1), turned to 180 degrees
- moved D21 0.29 mm to (111.3, 42.9)
- moved D23 0.13 mm to (76.6, 60.0)
- moved SW_POWER1 0.10 mm to (254.5, 50.3)
- turned D1 to 180 degrees
- turned D10 to 180 degrees
- turned D11 to 180 degrees
- turned D12 to 180 degrees
- turned D13 to 180 degrees
- turned D14 to 180 degrees
- turned D15 to 180 degrees
- turned D16 to 180 degrees
- turned D17 to 180 degrees
- turned D3 to 180 degrees
- turned D4 to 180 degrees
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Routing:
- net gnd: track 0.00 -> 194.1 mm, vias 0 -> 2
- net ROW1: track 0.00 -> 143.9 mm
- net COL0: track 0.00 -> 135.4 mm
- net vcc: track 0.00 -> 134.6 mm, vias 1 -> 3
- net ROW2: track 0.00 -> 133.1 mm
- net ROW0: track 0.00 -> 131.3 mm, vias 0 -> 1
- net IPD_CLK: track 0.00 -> 116.9 mm, vias 0 -> 3
- net IPD_DATA: track 0.00 -> 112.7 mm, vias 0 -> 2
- net COL1: track 0.00 -> 111.3 mm, vias 0 -> 6
- net IPD_RST: track 0.00 -> 108.6 mm, vias 0 -> 4
- net gnd_r: track 70.1 -> 173.1 mm
- net COL3: track 0.00 -> 91.4 mm, vias 0 -> 4
- net COL2: track 0.00 -> 86.5 mm, vias 1 -> 4
- net BT+: track 0.00 -> 81.9 mm, vias 0 -> 1
- net COL4: track 0.00 -> 76.3 mm, vias 0 -> 4
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- added copper zone on F.Cu, net gnd
- added copper zone on B.Cu, net gnd_r
- added copper zone on F.Cu, net gnd_r
Other:
- outline, holes or cut-outs redrawn
