File: roadrunner/roadrunner.kicad_pcb (KiCad board)
At the start: 2 copper layers, 246.8 x 97.3 mm, 88 parts, among them J1 Battery_conn, J2 battery_conn_r, J3 track_point_left, J4 niceview_left, J5 niceview_right, J6 track_point_right, J7 VIK_Left, J8 VIK_Right, SW1 SW_Push, SW10 SW_Push, SW10_r1 SW_Push, SW11 SW_Push, SW11_r1 SW_Push, SW12 SW_Push, SW12_r1 SW_Push, SW13 SW_Push, SW13_r1 SW_Push, SW14 SW_Push, SW14_r1 SW_Push, SW15 SW_Push, SW15_r1 SW_Push, SW16 SW_Push, SW16_r1 SW_Push, SW17 SW_Push, SW17_r1 SW_Push, SW1_r1 SW_Push, SW2 SW_Push, SW2_r1 SW_Push, SW3 SW_Push, SW3_r1 SW_Push, SW4 SW_Push, SW4_r1 SW_Push, SW5 SW_Push, SW5_r1 SW_Push, SW6 SW_Push, SW6_r1 SW_Push, SW7 SW_Push, SW7_r1 SW_Push, SW8 SW_Push, SW8_r1 SW_Push, SW9 SW_Push, SW9_r1 SW_Push, U1 ProMicro-kbd, U2 ProMicro-kbd

Commit message: chore: specify trackpoint model
Other:
- board text added: "t460s"
Changed lines of the file:
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@@
       (sketchpadsonfab false)
       (subtractmaskfromsilk false)
-      (outputformat 1)
+      (outputformat 5)
       (mirror false)
       (drillshape 0)
       (scaleselection 1)
-      (outputdirectory "roadrunner_v2_Gerber/")
+      (outputdirectory "seahorse_v2_gerber/")
     )
   )
@@
     (effects (font (size 2 2) (thickness 0.4) bold italic) (justify left bottom mirror))
   )
+  (gr_text "t460s" (at 182.42 38.82) (layer "B.SilkS")
+    (effects (font (size 1 1) (thickness 0.15)) (justify left bottom mirror))
+  )
   (gr_text "BT+" (at 250.0788 99.4807 60) (layer "B.SilkS")
     (effects (font (size 1 1) (thickness 0.15)) (justify mirror))
@@
     (effects (font (size 2 2) (thickness 0.15)) (justify left bottom mirror))
   )
+  (gr_text "t460s" (at 118.62 38.6) (layer "B.SilkS")
+    (effects (font (size 1 1) (thickness 0.15)) (justify left bottom mirror))
+  )
   (gr_text "BT+\n" (at 42.261025 101.988238 -60) (layer "B.SilkS")
